Commit message: [modify]

File: denso_robot_descriptions/vs087_description/vs087_and_mhand_with_phoxi/vs087_and_mhand_with_phoxi.urdf.xacro (robot description, xacro)
@@ -36,5 +36,5 @@
   <!-- Joint -->
   <joint name="joint_phoxi_left" type="fixed">
-    <origin xyz="1.620 2.200 1.400" rpy="-0.0411 0.2778 -2.231" />>
+    <origin xyz="1.500 2.220 1.400" rpy="-0.035 0.2778 -2.231" />>
     <!-- calibrated popsition -->
     <!-- <origin xyz="-0.686441 0.926263 0.761081" rpy="-3.12984 2.89395 2.18388" />> -->

Commit message: [modify] calibrated phoxi

File: denso_robot_descriptions/vs087_description/vs087_and_mhand_with_phoxi/vs087_and_mhand_with_phoxi.urdf.xacro (robot description, xacro)
@@ -36,7 +36,8 @@
   <!-- Joint -->
   <joint name="joint_phoxi_left" type="fixed">
+    <!-- initial position -->
     <origin xyz="1.500 2.220 1.400" rpy="-0.035 0.2778 -2.231" />>
     <!-- calibrated popsition -->
-    <!-- <origin xyz="-0.686441 0.926263 0.761081" rpy="-3.12984 2.89395 2.18388" />> -->
+    <!-- <origin xyz="1.26732 2.15934 1.59858" rpy="-3.00226 2.77424 0.944209" />> -->
     <parent link="world"/>
     <child link="phoxi_left_link"/>

Commit message: [modify] changed phoxi's fixed frame name

File: denso_robot_descriptions/vs087_description/vs087_and_mhand_with_phoxi/vs087_and_mhand_with_phoxi.urdf.xacro (robot description, xacro)
@@ -33,5 +33,6 @@
   <!-- Link -->
   <xacro:kinect2_link_box_v0 name="phoxi_left_link"/>
-  <link name="map"/> <!--  for playing bagfile 20181129 -->
+<!--   <link name="map"/>  for playing bagfile 2018.11.29 -->
+  <link name="phoxi_left_optical_frame"/> <!--  for playing bagfile 2018.12.17 -->
   <!-- Joint -->
   <joint name="joint_phoxi_left" type="fixed">
@@ -47,8 +48,9 @@
     <parent link="phoxi_left_link"/>
     <!-- <child link="kinect_left_rgb_optical_frame"/> -->
-    <child link="map"/>
+    <!-- <child link="map"/> -->
+    <child link="phoxi_left_optical_frame"/>
   </joint>
   <!-- Gazebo -->
-  <xacro:kinect_gazebo name="phoxi_left"/>
+<!--   <xacro:kinect_gazebo name="phoxi_left"/> -->
   <!-- add Kinect V2 -->
   <!-- kinect_right -->

Commit message: [modify] position of phoxi

File: denso_robot_descriptions/vs087_description/vs087_and_mhand_with_phoxi/vs087_and_mhand_with_phoxi.urdf.xacro (robot description, xacro)
@@ -38,7 +38,7 @@
   <joint name="joint_phoxi_left" type="fixed">
     <!-- initial position -->
-    <origin xyz="1.500 2.220 1.400" rpy="-0.035 0.2778 -2.231" />>
+    <!-- <origin xyz="1.500 2.220 1.400" rpy="-0.035 0.2778 -2.231" />> -->
     <!-- calibrated popsition -->
-    <!-- <origin xyz="1.26732 2.15934 1.59858" rpy="-3.00226 2.77424 0.944209" />> -->
+    <origin xyz="1.26732 2.15934 1.59858" rpy="-3.00226 2.77424 0.944209" />>
     <parent link="world"/>
     <child link="phoxi_left_link"/>
