Commit message: [add] center and left front kinect in the file

File: denso_robot_descriptions/vs087_description/vs087_and_mhand_with_kinect/vs087_and_mhand_with_kinect.urdf.xacro (robot description, xacro)
@@ -13,4 +13,22 @@
   <!-- add Kinect V2 -->
   <!-- kinect_center -->
+  <!-- Link -->
+  <xacro:kinect2_link_box_v0 name="kinect_center_link"/>
+  <link name="kinect_center_rgb_optical_frame"/>
+  <!-- Joint -->
+  <joint name="joint_kinect_center" type="fixed">
+    <origin xyz="0.8567 0.0762 0.9535" rpy="-0.0338 0.8795 3.0507" />
+    <parent link="world"/>
+    <child link="kinect_center_link"/>
+  </joint>
+  <joint name="joint_rgb_kinect_center" type="fixed">
+    <origin rpy="${M_PI/2} ${M_PI} ${M_PI/2}"/>
+    <parent link="kinect_center_link"/>
+    <child link="kinect_center_rgb_optical_frame"/>
+  </joint>
+  <!-- <!-\- Gazebo -\-> -->
+  <!-- <xacro:kinect_gazebo name="kinect_center"/> -->
+  <!-- add Kinect V2 -->
+  <!-- kinect_right_front -->
   <!-- Link -->
   <xacro:kinect2_link_box_v0 name="kinect_right_front_link"/>
@@ -32,3 +50,23 @@
   <!-- <!-\- Gazebo -\-> -->
   <!-- <xacro:kinect_gazebo name="kinect_right_front"/> -->
+  <!-- add Kinect V2 -->
+  <!-- kinect_left_front -->
+  <!-- Link -->
+  <xacro:kinect2_link_box_v0 name="kinect_left_front_link"/>
+  <link name="kinect_left_front_rgb_optical_frame"/>
+  <!-- Joint -->
+  <joint name="joint_kinect_left_front" type="fixed">
+    <!-- User calibration -->
+   <origin xyz="1.073 0.6515 0.6704" rpy="-0.0182 0.1578 -2.5882" />
+    <!-- calibrated popsition -->
+    <parent link="world"/>
+    <child link="kinect_left_front_link"/>
+  </joint>
+  <joint name="joint_rgb_kinect_left_front" type="fixed">
+    <origin rpy="${M_PI/2} ${M_PI} ${M_PI/2}"/>
+    <parent link="kinect_left_front_link"/>
+    <child link="kinect_left_front_rgb_optical_frame"/>
+  </joint>
+  <!-- <!-\- Gazebo -\-> -->
+  <!-- <xacro:kinect_gazebo name="kinect_left_front"/> -->
 </robot>

Commit message: [modify] changed position of kinect_center

File: denso_robot_descriptions/vs087_description/vs087_and_mhand_with_kinect/vs087_and_mhand_with_kinect.urdf.xacro (robot description, xacro)
@@ -18,5 +18,6 @@
   <!-- Joint -->
   <joint name="joint_kinect_center" type="fixed">
-    <origin xyz="0.8567 0.0762 0.9535" rpy="-0.0338 0.8795 3.0507" />
+    <!-- <origin xyz="0.8567 0.0762 0.9535" rpy="-0.0338 0.8795 3.0507" /> -->
+    <origin xyz="0.5500 0.05500 0.9000" rpy="-0.0338 0.8795 3.0507" />
     <parent link="world"/>
     <child link="kinect_center_link"/>

Commit message: [modify] erase kinect_right_front

File: denso_robot_descriptions/vs087_description/vs087_and_mhand_with_kinect/vs087_and_mhand_with_kinect.urdf.xacro (robot description, xacro)
@@ -19,5 +19,5 @@
   <joint name="joint_kinect_center" type="fixed">
     <!-- <origin xyz="0.8567 0.0762 0.9535" rpy="-0.0338 0.8795 3.0507" /> -->
-    <origin xyz="0.5500 0.05500 0.9000" rpy="-0.0338 0.8795 3.0507" />
+    <origin xyz="0.8567 0.0762 0.9535" rpy="-0.0338 0.8795 3.0507" />
     <parent link="world"/>
     <child link="kinect_center_link"/>
@@ -33,20 +33,21 @@
   <!-- kinect_right_front -->
   <!-- Link -->
-  <xacro:kinect2_link_box_v0 name="kinect_right_front_link"/>
+<!--   <xacro:kinect2_link_box_v0 name="kinect_right_front_link"/>
   <link name="kinect_right_front_rgb_optical_frame"/>
+ -->
   <!-- Joint -->
-  <joint name="joint_kinect_right_front" type="fixed">
+<!--   <joint name="joint_kinect_right_front" type="fixed"> -->
     <!-- User calibration -->
-    <origin xyz="1.1275 -0.7452 0.7101" rpy="0.0553 0.2057 2.5196" />
+<!--     <origin xyz="1.1275 -0.7452 0.7101" rpy="0.0553 0.2057 2.5196" /> -->
     <!-- calibrated popsition -->
     <!-- <origin xyz="-0.686441 -0.926263 0.761081" rpy="-0.0233 0.3223 0.481" />> -->
-    <parent link="world"/>
+<!--     <parent link="world"/>
     <child link="kinect_right_front_link"/>
-  </joint>
-  <joint name="joint_rgb_kinect_right_front" type="fixed">
+  </joint> -->
+<!--   <joint name="joint_rgb_kinect_right_front" type="fixed">
     <origin rpy="${M_PI/2} ${M_PI} ${M_PI/2}"/>
     <parent link="kinect_right_front_link"/>
     <child link="kinect_right_front_rgb_optical_frame"/>
-  </joint>
+  </joint> -->
   <!-- <!-\- Gazebo -\-> -->
   <!-- <xacro:kinect_gazebo name="kinect_right_front"/> -->
@@ -59,6 +60,7 @@
   <joint name="joint_kinect_left_front" type="fixed">
     <!-- User calibration -->
-   <origin xyz="1.073 0.6515 0.6704" rpy="-0.0182 0.1578 -2.5882" />
+    <origin xyz="1.073 0.6515 0.6704" rpy="-0.0389 0.3127 -2.6041" />
     <!-- calibrated popsition -->
+    <!-- <origin xyz="0.958735 0.71587 0.756947" rpy="3.11561 2.75096 0.663577" /> -->
     <parent link="world"/>
     <child link="kinect_left_front_link"/>

Commit message: [modify] leave only kinect_right_front

File: denso_robot_descriptions/vs087_description/vs087_and_mhand_with_kinect/vs087_and_mhand_with_kinect.urdf.xacro (robot description, xacro)
@@ -14,11 +14,12 @@
   <!-- kinect_center -->
   <!-- Link -->
-  <xacro:kinect2_link_box_v0 name="kinect_center_link"/>
+<!--   <xacro:kinect2_link_box_v0 name="kinect_center_link"/>
   <link name="kinect_center_rgb_optical_frame"/>
+ -->
   <!-- Joint -->
-  <joint name="joint_kinect_center" type="fixed">
-    <!-- <origin xyz="0.8567 0.0762 0.9535" rpy="-0.0338 0.8795 3.0507" /> -->
-    <origin xyz="0.5500 0.05500 0.9000" rpy="-0.0338 0.8795 3.0507" />
-    <parent link="world"/>
+<!--   <joint name="joint_kinect_center" type="fixed">
+    <origin xyz="0.8567 0.0762 0.9535" rpy="-0.0338 0.8795 3.0507" />
+ --><!-- <origin xyz="0.5500 0.05500 0.9000" rpy="-0.0338 0.8795 3.0507" /> -->
+<!--     <parent link="world"/>
     <child link="kinect_center_link"/>
   </joint>
@@ -28,4 +29,5 @@
     <child link="kinect_center_rgb_optical_frame"/>
   </joint>
+ -->
   <!-- <!-\- Gazebo -\-> -->
   <!-- <xacro:kinect_gazebo name="kinect_center"/> -->
@@ -54,12 +56,13 @@
   <!-- kinect_left_front -->
   <!-- Link -->
-  <xacro:kinect2_link_box_v0 name="kinect_left_front_link"/>
+<!--   <xacro:kinect2_link_box_v0 name="kinect_left_front_link"/>
   <link name="kinect_left_front_rgb_optical_frame"/>
+ -->
   <!-- Joint -->
-  <joint name="joint_kinect_left_front" type="fixed">
-    <!-- User calibration -->
-   <origin xyz="1.073 0.6515 0.6704" rpy="-0.0182 0.1578 -2.5882" />
-    <!-- calibrated popsition -->
-    <parent link="world"/>
+<!--   <joint name="joint_kinect_left_front" type="fixed">
+ -->    <!-- User calibration -->
+<!--    <origin xyz="1.073 0.6515 0.6704" rpy="-0.0182 0.1578 -2.5882" />
+ -->    <!-- calibrated popsition -->
+<!--     <parent link="world"/>
     <child link="kinect_left_front_link"/>
   </joint>
@@ -69,5 +72,5 @@
     <child link="kinect_left_front_rgb_optical_frame"/>
   </joint>
-  <!-- <!-\- Gazebo -\-> -->
+ -->  <!-- <!-\- Gazebo -\-> -->
   <!-- <xacro:kinect_gazebo name="kinect_left_front"/> -->
 </robot>

Commit message: [modify] appeared kinect_center

File: denso_robot_descriptions/vs087_description/vs087_and_mhand_with_kinect/vs087_and_mhand_with_kinect.urdf.xacro (robot description, xacro)
@@ -14,8 +14,8 @@
   <!-- kinect_center -->
   <!-- Link -->
-<!--   <xacro:kinect2_link_box_v0 name="kinect_center_link"/>
-  <link name="kinect_center_rgb_optical_frame"/> -->
+  <xacro:kinect2_link_box_v0 name="kinect_center_link"/>
+  <link name="kinect_center_rgb_optical_frame"/>
   <!-- Joint -->
-<!--   <joint name="joint_kinect_center" type="fixed">
+  <joint name="joint_kinect_center" type="fixed">
     <origin xyz="0.8567 0.0762 0.9535" rpy="-0.0338 0.8795 3.0507" />
   <origin xyz="0.5500 0.05500 0.9000" rpy="-0.0338 0.8795 3.0507" />
@@ -27,5 +27,5 @@
     <parent link="kinect_center_link"/>
     <child link="kinect_center_rgb_optical_frame"/>
-  </joint> -->
+  </joint>
   <!-- <!-\- Gazebo -\-> -->
   <!-- <xacro:kinect_gazebo name="kinect_center"/> -->
@@ -54,12 +54,15 @@
   <!-- kinect_left_front -->
   <!-- Link -->
- <!--  <xacro:kinect2_link_box_v0 name="kinect_left_front_link"/>
-  <link name="kinect_left_front_rgb_optical_frame"/> -->
+  <xacro:kinect2_link_box_v0 name="kinect_left_front_link"/>
+  <link name="kinect_left_front_rgb_optical_frame"/>
   <!-- Joint -->
-<!--   <joint name="joint_kinect_left_front" type="fixed"> -->
+  <joint name="joint_kinect_left_front" type="fixed">
     <!-- User calibration -->
-<!--     <origin xyz="1.073 0.6515 0.6704" rpy="-0.0182 0.1578 -2.5882" /> -->
+    <!-- <origin xyz="1.073 0.6515 0.6704" rpy="-0.0182 0.1578 -2.5882" /> -->
+	<origin xyz="1.073 0.6515 0.6704" rpy="-0.0389 0.3127 -2.6041" />
     <!-- calibrated popsition -->
-<!--     <parent link="world"/>
+    <!-- <origin xyz="0.958735 0.71587 0.756947" rpy="3.11561 2.75096 0.663577" /> -->
+    <!-- calibrated popsition -->
+    <parent link="world"/>
     <child link="kinect_left_front_link"/>
   </joint>
@@ -68,6 +71,6 @@
     <parent link="kinect_left_front_link"/>
     <child link="kinect_left_front_rgb_optical_frame"/>
-  </joint> -->
-  <!-- <!-\- Gazebo -\-> -->
-  <!-- <xacro:kinect_gazebo name="kinect_left_front"/> -->
+  </joint>
+  <!-- Gazebo -->
+  <xacro:kinect_gazebo name="kinect_left_front"/>
 </robot>

Commit message: [modify] changed the frame position

File: denso_robot_descriptions/vs087_description/vs087_and_mhand_with_kinect/vs087_and_mhand_with_kinect.urdf.xacro (robot description, xacro)
@@ -14,8 +14,8 @@
   <!-- kinect_center -->
   <!-- Link -->
-  <xacro:kinect2_link_box_v0 name="kinect_center_link"/>
+   <xacro:kinect2_link_box_v0 name="kinect_center_link"/>
   <link name="kinect_center_rgb_optical_frame"/>
   <!-- Joint -->
-  <joint name="joint_kinect_center" type="fixed">
+   <joint name="joint_kinect_center" type="fixed">
     <origin xyz="0.8567 0.0762 0.9535" rpy="-0.0338 0.8795 3.0507" />
   <origin xyz="0.5500 0.05500 0.9000" rpy="-0.0338 0.8795 3.0507" />
@@ -33,10 +33,10 @@
   <!-- kinect_right_front -->
   <!-- Link -->
-  <xacro:kinect2_link_box_v0 name="kinect_right_front_link"/>
+   <xacro:kinect2_link_box_v0 name="kinect_right_front_link"/>
   <link name="kinect_right_front_rgb_optical_frame"/>
   <!-- Joint -->
-  <joint name="joint_kinect_right_front" type="fixed">
+   <joint name="joint_kinect_right_front" type="fixed">
     <!-- User calibration -->
-    <origin xyz="1.1275 -0.7452 0.7101" rpy="0.0553 0.2057 2.5196" />
+     <origin xyz="1.1275 -0.7452 0.7101" rpy="0.0553 0.2057 2.5196" />
     <!-- calibrated popsition -->
     <!-- <origin xyz="-0.686441 -0.926263 0.761081" rpy="-0.0233 0.3223 0.481" />> -->
@@ -59,9 +59,11 @@
   <joint name="joint_kinect_left_front" type="fixed">
     <!-- User calibration -->
-    <!-- <origin xyz="1.073 0.6515 0.6704" rpy="-0.0182 0.1578 -2.5882" /> -->
-	<origin xyz="1.073 0.6515 0.6704" rpy="-0.0389 0.3127 -2.6041" />
+    <origin xyz="1.073 0.6515 0.6704" rpy="-0.0182 0.1578 -2.5882" />
+  <!-- 	<origin xyz="1.073 0.6515 0.6704" rpy="-0.0389 0.3127 -2.6041" /> -->
+  <!-- <origin xyz="0.9631 0.7215 0.7402" rpy="-0.0037 0.3558 -2.4763" /> -->
     <!-- calibrated popsition -->
     <!-- <origin xyz="0.958735 0.71587 0.756947" rpy="3.11561 2.75096 0.663577" /> -->
-    <!-- calibrated popsition -->
+    <!-- <origin xyz="0.960046 0.719561 0.73759" rpy="3.1379 2.7858 0.6656" /> -->
+    <!-- <origin xyz="0.95349 0.726311 0.74168" rpy="-3.13512 2.76347 0.683613" /> -->
     <parent link="world"/>
     <child link="kinect_left_front_link"/>

Commit message: [modify] シミュレーション用のあれこれの追加

File: denso_robot_descriptions/vs087_description/vs087_and_mhand_with_kinect/vs087_and_mhand_with_kinect.urdf.xacro (robot description, xacro)
@@ -60,6 +60,6 @@
     <!-- User calibration -->
     <origin xyz="1.073 0.6515 0.6704" rpy="-0.0182 0.1578 -2.5882" />
-  <!-- 	<origin xyz="1.073 0.6515 0.6704" rpy="-0.0389 0.3127 -2.6041" /> -->
-  <!-- <origin xyz="0.9631 0.7215 0.7402" rpy="-0.0037 0.3558 -2.4763" /> -->
+    <!-- <origin xyz="1.073 0.6515 0.6704" rpy="-0.0389 0.3127 -2.6041" /> -->
+    <!-- <origin xyz="0.9631 0.7215 0.7402" rpy="-0.0037 0.3558 -2.4763" /> -->
     <!-- calibrated popsition -->
     <!-- <origin xyz="0.958735 0.71587 0.756947" rpy="3.11561 2.75096 0.663577" /> -->
